Commit message: reduced image sizes

File: packages/robot_description/urdf/robot.urdf.xacro (robot description, xacro)
@@ -4,9 +4,9 @@
     <xacro:property name="mesh_prefix" value="package://robot_description/meshes" />
     <!-- Wheel properties -->
-    <xacro:property name="wheel_radius" value="0.03" />
-    <xacro:property name="wheel_width" value="0.02" />
-    <xacro:property name="wheel_x_offset" value="0.06" />
+    <xacro:property name="wheel_radius" value="0.033" />
+    <xacro:property name="wheel_width" value="0.03" />
+    <xacro:property name="wheel_x_offset" value="0.055" />
     <xacro:property name="wheel_y_offset" value="0.105" />
-    <xacro:property name="wheel_z_offset" value="-0.05" />
+    <xacro:property name="wheel_z_offset" value="-0.0784" />
     <!-- ===================== LINKS ===================== -->
     <!-- BASE FOOTPRINT -->
@@ -27,5 +27,5 @@
             <origin xyz="0 0 0" rpy="0 0 0" />
             <geometry>
-                <box size="0.02 0.02 0.01" />
+                <box size="0.03 0.03 0.01" />
             </geometry>
         </visual>
@@ -36,5 +36,5 @@
             <origin xyz="0 0 0" rpy="0 0 0" />
             <geometry>
-                <cylinder radius="0.038" length="0.04" />
+                <cylinder radius="0.035" length="0.02368" />
             </geometry>
         </visual>
@@ -84,5 +84,5 @@
         <parent link="base_link" />
         <child link="imu_link" />
-        <origin xyz="0.0 0.0 0.05" rpy="0 0 0" />
+        <origin xyz="-0.044 0.006 -0.0575" rpy="0 0 0" />
     </joint>
     <!-- RPLIDAR JOINT -->
@@ -90,5 +90,5 @@
         <parent link="base_link" />
         <child link="lidar_link" />
-        <origin xyz="0.0 0.0 0.12" rpy="0 0 0" />
+        <origin xyz="0.0 0.0 0.0" rpy="0 0 0" />
     </joint>
     <!-- WHEEL JOINTS (continuous for driven wheels) -->
