Commit message: revise image optimization

File: docker_ws/src/robot_description/urdf/robot.urdf.xacro (robot description, xacro)
@@ -2,5 +2,5 @@
 <robot xmlns:xacro="http://www.ros.org/wiki/xacro" name="robot">
     <!-- Mesh path prefix -->
-    <xacro:property name="mesh_prefix" value="package://robot_description/meshes" />
+    <!-- <xacro:property name="mesh_prefix" value="package://robot_description/meshes" /> -->
     <!-- Wheel properties -->
     <xacro:property name="wheel_radius" value="0.033" />
@@ -15,10 +15,10 @@
     <!-- BASE LINK -->
     <link name="base_link">
-        <visual>
-            <origin xyz="0 0 0" rpy="0 0 0" />
+        <!-- <visual>
+            <origin xyz="0 -0.072 0" rpy="0 0 0" />
             <geometry>
                 <mesh filename="${mesh_prefix}/robot.obj" />
             </geometry>
-        </visual>
+        </visual> -->
     </link>
     <!-- IMU LINK -->

Commit message: params update

File: docker_ws/src/robot_description/urdf/robot.urdf.xacro (robot description, xacro)
@@ -90,5 +90,5 @@
         <parent link="base_link" />
         <child link="lidar_link" />
-        <origin xyz="0.0 0.0 0.0" rpy="0 0 0" />
+        <origin xyz="0.0 0.0 0.0" rpy="0 0 ${pi}" />
     </joint>
     <!-- WHEEL JOINTS (continuous for driven wheels) -->

Commit message: imu datasets + calibration

File: docker_ws/src/robot_description/urdf/robot.urdf.xacro (robot description, xacro)
@@ -84,5 +84,5 @@
         <parent link="base_link" />
         <child link="imu_link" />
-        <origin xyz="-0.044 0.006 -0.0575" rpy="0 0 0" />
+        <origin xyz="-0.044 0.006 -0.0575" rpy="0 0 ${pi}" />
     </joint>
     <!-- RPLIDAR JOINT -->
